File: UINIO-USB-Serial.kicad_pcb (KiCad board)
At the start: 2 copper layers, 0 parts

Commit message: Complete the schematic test.
Parts:
- added C1: 0.1uF, Capacitor_SMD:C_0402_1005Metric, F.Cu at (153.5, 85.1)
- added C2: 0.1uF, Capacitor_SMD:C_0402_1005Metric, F.Cu at (257.6, 74.6)
- added C3: 20pF, Capacitor_SMD:C_0402_1005Metric, F.Cu at (153.5, 89.0)
- added C4: 20pF, Capacitor_SMD:C_0402_1005Metric, F.Cu at (153.5, 91.0)
- added C5: 0.1uF, Capacitor_SMD:C_0402_1005Metric, F.Cu at (153.5, 92.9)
- added C6: 0.1uF, Capacitor_SMD:C_0402_1005Metric, F.Cu at (257.6, 82.5)
- added C7: 0.1uF, Capacitor_SMD:C_0402_1005Metric, F.Cu at (257.6, 84.5)
- added C8: 1uF, Capacitor_SMD:C_0603_1608Metric, F.Cu at (142.5, 86.0)
- added C9: 1uF, Capacitor_SMD:C_0603_1608Metric, F.Cu at (142.5, 88.5)
- added D1: LED Blue, LED_SMD:LED_0603_1608Metric, F.Cu at (177.9, 84.2)
- added D2: LED_Red, LED_SMD:LED_0603_1608Metric, F.Cu at (224.5, 102.0)
- added J1: Conn_01x10_Pin, Connector_PinHeader_2.54mm:PinHeader_1x10_P2.54mm_Vertical, F.Cu at (138.2, 70.5)
- added J10: Conn_01x07_Pin, Connector_PinHeader_2.54mm:PinHeader_1x07_P2.54mm_Vertical, F.Cu at (174.3, 108.9)
- added J2: Conn_01x06_Pin, Connector_PinHeader_2.54mm:PinHeader_1x06_P2.54mm_Vertical, F.Cu at (214.8, 86.2)
- added J3: Conn_01x07_Pin, Connector_PinHeader_2.54mm:PinHeader_1x07_P2.54mm_Vertical, F.Cu at (138.2, 108.9)
- added J4: Conn_01x04_Pin, Connector_PinHeader_2.54mm:PinHeader_1x04_P2.54mm_Vertical, F.Cu at (252.3, 90.5)
- added J5: Conn_01x07_Pin, Connector_PinHeader_2.54mm:PinHeader_1x07_P2.54mm_Vertical, F.Cu at (174.3, 70.5)
- added J6: Conn_01x04_Pin, Connector_PinHeader_2.54mm:PinHeader_1x04_P2.54mm_Vertical, F.Cu at (160.1, 108.9)
- added J7: Conn_01x03_Pin, Connector_PinHeader_2.54mm:PinHeader_1x03_P2.54mm_Vertical, F.Cu at (186.3, 86.7)
- added J8: Conn_01x03_Pin, Connector_PinHeader_2.54mm:PinHeader_1x03_P2.54mm_Vertical, F.Cu at (191.0, 86.7)
- added J9: Conn_01x04_Pin, Connector_PinHeader_2.54mm:PinHeader_1x04_P2.54mm_Vertical, F.Cu at (261.6, 90.5)
- added R1: 4.7K, Resistor_SMD:R_0402_1005Metric, F.Cu at (156.4, 85.1)
- added R10: 4.7K, Resistor_SMD:R_0402_1005Metric, F.Cu at (189.0, 80.4)
- added R11: 4.7K, Resistor_SMD:R_0402_1005Metric, F.Cu at (189.0, 82.4)
- added R2: 5.1K, Resistor_SMD:R_0402_1005Metric, F.Cu at (260.5, 74.6)
- added R3: 5.1K, Resistor_SMD:R_0402_1005Metric, F.Cu at (260.5, 76.6)
- added R4: 10K, Resistor_SMD:R_0402_1005Metric, F.Cu at (260.5, 78.6)
- added R5: 10K, Resistor_SMD:R_0402_1005Metric, F.Cu at (260.5, 80.6)
- added R6: 2K, Resistor_SMD:R_0402_1005Metric, F.Cu at (156.4, 95.0)
- added R7: 10K, Resistor_SMD:R_0402_1005Metric, F.Cu at (263.4, 72.7)
- added R8: 10K, Resistor_SMD:R_0402_1005Metric, F.Cu at (263.4, 74.6)
- added R9: 2K, Resistor_SMD:R_0402_1005Metric, F.Cu at (263.4, 76.6)
- added U1: I2C-24-EEPROM-SOIC8, Package_SO:SOIC-8_3.9x4.9mm_P1.27mm, F.Cu at (234.9, 91.4)
- added U2: CH347T, Uinio:TSSOP-20_L6.5-W4.4-P0.65-LS6.4-BL, F.Cu at (164.2, 88.0)
- added U3: SPI-25-Flash-SOIC8, Package_SO:SOIC-8_5.23x5.23mm_P1.27mm, F.Cu at (232.1, 75.4)
- added U4: I2C-24-EEPROM-TSSOP8, Package_SO:TSSOP-8_4.4x3mm_P0.65mm, F.Cu at (221.6, 95.8)
- added U5: ME6211C33M5G, Uinio:SOT-23-5_L3.0-W1.7-P0.95-LS2.8-BR, F.Cu at (142.8, 92.0)
- added USB1: USB_Type_C_16Pin, Uinio:USB-C-SMD_TYPEC-304J-BCP16, F.Cu at (129.1, 89.4)
- added Y1: 8MHz, Crystal:Crystal_SMD_3225-4Pin_3.2x2.5mm, F.Cu at (173.2, 85.2)

Commit message: Finish PCB layout.
Parts:
- removed C7: 0.1uF, Capacitor_SMD:C_0402_1005Metric
- removed C8, C9: 1uF, Capacitor_SMD:C_0603_1608Metric
- removed J10: Conn_01x07_Pin, Connector_PinHeader_2.54mm:PinHeader_1x07_P2.54mm_Vertical
- removed J8: Conn_01x03_Pin, Connector_PinHeader_2.54mm:PinHeader_1x03_P2.54mm_Vertical
- removed J9: Conn_01x04_Pin, Connector_PinHeader_2.54mm:PinHeader_1x04_P2.54mm_Vertical
- removed R10, R11: 4.7K, Resistor_SMD:R_0402_1005Metric
- removed U3: SPI-25-Flash-SOIC8, Package_SO:SOIC-8_5.23x5.23mm_P1.27mm
- removed U4: I2C-24-EEPROM-TSSOP8, Package_SO:TSSOP-8_4.4x3mm_P0.65mm
- removed U5: ME6211C33M5G, Uinio:SOT-23-5_L3.0-W1.7-P0.95-LS2.8-BR
- added HOLE**: Hole-1mm, Uinio:Hole-1mm, F.Cu at (93.2, 48.0)
- added HOLE**: Hole-1mm, Uinio:Hole-1mm, F.Cu at (144.8, 62.3)
- added HOLE**: Hole-1mm, Uinio:Hole-1mm, F.Cu at (144.8, 48.0)
- added HOLE**: Hole-1mm, Uinio:Hole-1mm, F.Cu at (93.2, 62.3)
- added HOLE**: Hole-1mm, Uinio:Hole-1mm, F.Cu at (122.8, 42.4)
- C2: value 0.1uF -> 20pF
- C3: value 20pF -> 0.1uF
- C5, C6: value 0.1uF -> 1uF; footprint Capacitor_SMD:C_0402_1005Metric -> Capacitor_SMD:C_0603_1608Metric
- J1: value Conn_01x10_Pin -> Conn_01x07_Pin; footprint Connector_PinHeader_2.54mm:PinHeader_1x10_P2.54mm_Vertical -> Connector_PinHeader_2.54mm:PinHeader_1x07_P2.54mm_Vertical
- J2: value Conn_01x06_Pin -> Conn_01x10_Pin; footprint Connector_PinHeader_2.54mm:PinHeader_1x06_P2.54mm_Vertical -> Connector_PinHeader_2.54mm:PinHeader_1x10_P2.54mm_Vertical
- J3: value Conn_01x07_Pin -> Conn_01x04_Pin; footprint Connector_PinHeader_2.54mm:PinHeader_1x07_P2.54mm_Vertical -> Connector_PinHeader_2.54mm:PinHeader_1x04_P2.54mm_Vertical
- J4: value Conn_01x04_Pin -> Conn_01x07_Pin; footprint Connector_PinHeader_2.54mm:PinHeader_1x04_P2.54mm_Vertical -> Connector_PinHeader_2.54mm:PinHeader_1x07_P2.54mm_Vertical
- J5: value Conn_01x07_Pin -> 排针1; footprint Connector_PinHeader_2.54mm:PinHeader_1x07_P2.54mm_Vertical -> Connector_PinHeader_2.54mm:PinHeader_1x03_P2.54mm_Vertical
- J6: value Conn_01x04_Pin -> 排针2; footprint Connector_PinHeader_2.54mm:PinHeader_1x04_P2.54mm_Vertical -> Connector_PinHeader_2.54mm:PinHeader_1x03_P2.54mm_Vertical
- J7: value Conn_01x03_Pin -> Conn_01x07_Pin; footprint Connector_PinHeader_2.54mm:PinHeader_1x03_P2.54mm_Vertical -> Connector_PinHeader_2.54mm:PinHeader_1x07_P2.54mm_Vertical
- R2, R3: footprint Resistor_SMD:R_0402_1005Metric -> Resistor_SMD:R_0603_1608Metric
- R4, R5: value 10K -> 2K
- R6, R9: value 2K -> 4.7K
- R7, R8: value 10K -> 4.7K
- U1: value I2C-24-EEPROM-SOIC8 -> CH347T; footprint Package_SO:SOIC-8_3.9x4.9mm_P1.27mm -> Uinio:TSSOP-20_L6.5-W4.4-P0.65-LS6.4-BL
- U2: value CH347T -> ME6211C33M5G; footprint Uinio:TSSOP-20_L6.5-W4.4-P0.65-LS6.4-BL -> Uinio:SOT-23-5_L3.0-W1.7-P0.95-LS2.8-BR
- moved R3 156.1 mm to (106.5, 51.2), turned to 90 degrees
- moved R2 153.8 mm to (108.5, 51.2), turned to -90 degrees
- moved R5 151.1 mm to (112.2, 51.7), turned to -90 degrees
- moved C6 147.4 mm to (112.0, 59.5), turned to 90 degrees
- moved C2 140.3 mm to (120.1, 46.6), turned to -90 degrees
- moved R7 133.5 mm to (131.6, 51.7), turned to 180 degrees
- moved J4 133.4 mm to (127.8, 42.4), turned to 90 degrees
- moved R9 133.1 mm to (131.6, 58.3), turned to 180 degrees
- moved R8 132.6 mm to (131.6, 59.8), turned to 180 degrees
- moved R4 131.1 mm to (131.6, 54.7)
- moved J2 127.7 mm to (94.8, 42.4), turned to 90 degrees
- moved D2 124.8 mm to (110.5, 51.2), turned to -90 degrees
- moved U1 118.0 mm to (122.7, 55.1)
- moved J7 78.6 mm to (110.1, 67.8), turned to -90 degrees
- moved Y1 63.1 mm to (122.7, 47.4), turned to 180 degrees
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Connections:
- C1 pad 1: Net-(U2-RST#) -> Net-(U1-RST#)
- C2 pad 1: /EEPROM-SOIC8-GND -> GND
- C2 pad 2: /EEPROM-SOIC8-3.3V -> Net-(U1-XO)
- C3 pad 1: GND -> /VDD_3.3V
- C3 pad 2: Net-(U2-XO) -> GND
- C4 pad 2: Net-(U2-XI) -> Net-(U1-XI)
- C5 pad 1: /VDD_3.3V -> GND
- C5 pad 2: GND -> /VDD_5V
- C6 pad 1: /Flash-SOIC8-GND -> GND
- C6 pad 2: /Flash-SOIC8-3.3V -> /VDD_3.3V
- J1 pad 2: /CTS0/SCK/TCK -> /DSR0/CS0/TMS
- J1 pad 3: /JTAG_TDI -> /DTR0/IO5
- J1 pad 4: /I2C_SDA -> /CTS0/SCK/TCK
- J1 pad 6: /DTR0/IO5 -> /JTAG_TDI
- J1 pad 7: /DSR0/CS0/TMS -> /VDD_3.3V
- J2 pad 1: /Flash-SOIC8-GND -> GND
- J2 pad 2: /Flash-SOIC8-MISO -> /JTAG_TDI
- J2 pad 3: /Flash-SOIC8-MOSI -> /I2C_SDA
- J2 pad 4: /Flash-SOIC8-CLK -> /CTS0/SCK/TCK
- J2 pad 5: /Flash-SOIC8-CS -> /JTAG_TDO
- J2 pad 6: /Flash-SOIC8-3.3V -> /DTR0/IO5
- J3 pad 1: GND -> /VDD_3.3V
- J3 pad 2: /CTS1/IO6 -> /I2C_SDA
- J3 pad 3: /TXD1 -> /I2C_SCL
- J3 pad 4: /RXD1 -> GND
- J4 pad 1: /EEPROM-SOIC8-3.3V -> GND
- J4 pad 2: Net-(J4-Pin_2) -> /TXD1
- J4 pad 3: Net-(J4-Pin_3) -> /RXD1
- J4 pad 4: /EEPROM-SOIC8-GND -> /CTS1/IO6
- J5 pad 1: GND -> Net-(J5-Pin_1)
- J5 pad 2: /DSR0/CS0/TMS -> /RTS1/IO7
- J5 pad 3: /DTR0/IO5 -> Net-(J5-Pin_3)
- J6 pad 1: /VDD_3.3V -> Net-(J6-Pin_1)
- J6 pad 2: /I2C_SDA -> /DTR1
- J6 pad 3: /I2C_SCL -> Net-(J6-Pin_3)
- J7 pad 1: Net-(J7-Pin_1) -> GND
- J7 pad 2: /P1 -> /CTS0/SCK/TCK
- J7 pad 3: unconnected-(J7-Pin_3-Pad3) -> /DSR0/CS0/TMS
- R1 pad 2: Net-(U2-RST#) -> Net-(U1-RST#)
- R4 pad 1: Net-(J4-Pin_3) -> Net-(D1-A)
- R4 pad 2: /EEPROM-SOIC8-3.3V -> /VDD_3.3V
- R5 pad 1: Net-(J4-Pin_2) -> Net-(D2-A)
- R5 pad 2: /EEPROM-SOIC8-3.3V -> /VDD_3.3V
- R6 pad 1: Net-(D1-A) -> Net-(J5-Pin_1)
- R6 pad 2: /VDD_3.3V -> GND
- R7 pad 1: Net-(J9-Pin_3) -> Net-(J6-Pin_1)
- R7 pad 2: /EEPROM-TSSOP8-3.3V -> GND
- R8 pad 1: Net-(J9-Pin_2) -> Net-(J5-Pin_3)
- R8 pad 2: /EEPROM-TSSOP8-3.3V -> /VDD_3.3V
- R9 pad 1: Net-(D2-A) -> Net-(J6-Pin_3)
- U1 pad 1: /EEPROM-SOIC8-GND -> Net-(U1-RST#)
- U1 pad 2: /EEPROM-SOIC8-GND -> /CTS1/IO6
- U1 pad 3: /EEPROM-SOIC8-GND -> /TXD1
- U1 pad 4: /EEPROM-SOIC8-GND -> /RXD1
- U1 pad 5: Net-(J4-Pin_2) -> /DSR0/CS0/TMS
- U1 pad 6: Net-(J4-Pin_3) -> /CTS0/SCK/TCK
- U1 pad 7: /EEPROM-SOIC8-GND -> /JTAG_TDO
- U1 pad 8: /EEPROM-SOIC8-3.3V -> /JTAG_TDI
- U2 pad 1: Net-(U2-RST#) -> /VDD_5V
- U2 pad 2: /CTS1/IO6 -> GND
- U2 pad 3: /TXD1 -> /VDD_5V
- U2 pad 4: /RXD1 -> unconnected-(U2-NC-Pad4)
- U2 pad 5: /DSR0/CS0/TMS -> /VDD_3.3V
- Y1 pad 1: Net-(U2-XO) -> Net-(U1-XO)
- Y1 pad 2: Net-(U2-XI) -> GND
- Y1 pad 3: (no net) -> Net-(U1-XI)
- Y1 pad 4: (no net) -> GND
Other:
- board outline added: 55.3 x 28.1 mm
- board text added: "3V3"
- board text added: "CH347T"
- board text added: "CS0"
- board text added: "CS1"
- board text added: "CTS"
- board text added: "DCD"
- board text added: "DSR"
- board text added: "DTR"
- board text added: "GND"
- board text added: "MISO"
- board text added: "MOSI"
- board text added: "RI"
- board text added: "RST"
- board text added: "RTS"
- board text added: "RXD"
- board text added: "SCK"
- board text added: "SCL"
- board text added: "SDA"
- board text added: "TCK"
- board text added: "TDI"
- board text added: "TDO"
- board text added: "TMS"
- board text added: "TXD"
- board text added: "UinIO.com"
- board text added: "低 电 平"
- board text added: "高 电 平"

Commit message: Finish PCB layout.
Parts:
- moved J6 0.97 mm to (141.9, 52.6)
- moved J5 0.97 mm to (138.5, 52.6)
- moved C5 0.26 mm to (106.2, 59.5)
- moved D2 0.26 mm to (110.2, 51.2)
- moved C6 0.25 mm to (111.8, 59.5)
- moved R2 0.25 mm to (108.2, 51.2)
- moved R3 0.25 mm to (106.2, 51.2)
- moved R5 0.25 mm to (111.9, 51.7)
- moved U2 0.25 mm to (109.0, 59.6)
- moved C2 0.16 mm to (120.2, 46.7)
- moved C4 0.16 mm to (125.3, 46.7)
- moved C1 0.12 mm to (119.9, 61.6)
- moved U1 0.12 mm to (122.8, 55.1)
- moved Y1 0.12 mm to (122.8, 47.4)
- moved R1 0.12 mm to (121.5, 61.6)
Other:
- board text added: "UINIO-USB-Serial"
- board text added: "Version 1.0.0"
- board text added: "排针 P1"
- board text added: "排针 P2"

Commit message: Finish PCB layout.
Parts:
- moved R3 58.2 mm to (143.5, 96.0)
- moved R9 58.2 mm to (166.9, 104.5)
- moved D1 57.1 mm to (166.4, 101.3)
- moved J3 57.0 mm to (158.1, 112.6)
- moved R1 57.0 mm to (156.8, 106.5)
- moved HOLE** 57.0 mm to (128.6, 92.8)
- moved J5 57.0 mm to (173.8, 97.4)
- moved J6 57.0 mm to (177.2, 97.4)
- moved Y1 57.0 mm to (158.1, 92.2), turned to -90 degrees
- moved C1 57.0 mm to (155.2, 106.4)
- moved C2 57.0 mm to (155.5, 91.5), turned to 90 degrees
- moved C3 57.0 mm to (166.9, 95.0)
- moved C4 57.0 mm to (160.7, 91.5), turned to -90 degrees
- moved C5 57.0 mm to (141.5, 104.3)
- moved HOLE** 57.0 mm to (180.1, 107.1)
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Connections:
- J1 pad 3: /DTR0/IO5 -> /CTS0/SCK/TCK
- J1 pad 4: /CTS0/SCK/TCK -> /JTAG_TDO
- J1 pad 5: /JTAG_TDO -> /JTAG_TDI
- J1 pad 6: /JTAG_TDI -> /DTR0/IO5
- J2 pad 2: /JTAG_TDI -> /DTR0/IO5
- J2 pad 3: /I2C_SDA -> /JTAG_TDI
- J2 pad 4: /CTS0/SCK/TCK -> /JTAG_TDO
- J2 pad 5: /JTAG_TDO -> /CTS0/SCK/TCK
- J2 pad 6: /DTR0/IO5 -> /DSR0/CS0/TMS
- J2 pad 7: /DSR0/CS0/TMS -> /DCD0/IO4
- J2 pad 8: /I2C_SCL -> /I2C_SDA
- J2 pad 9: /DCD0/IO4 -> /I2C_SCL
- J3 pad 2: /I2C_SDA -> /I2C_SCL
- J3 pad 3: /I2C_SCL -> /I2C_SDA
- J4 pad 2: /TXD1 -> /RTS1/IO7
- J4 pad 3: /RXD1 -> /CTS1/IO6
- J4 pad 4: /CTS1/IO6 -> /TXD1
- J4 pad 5: /RTS1/IO7 -> /RXD1
- J7 pad 2: /CTS0/SCK/TCK -> /DSR0/CS0/TMS
- J7 pad 3: /DSR0/CS0/TMS -> /CTS0/SCK/TCK
- J7 pad 4: /JTAG_TDI -> /JTAG_TDO
- J7 pad 5: /JTAG_TDO -> /JTAG_TDI
Routing:
- net /VDD_3.3V: track 0.00 -> 149.9 mm, vias 0 -> 5
- net /DTR0/IO5: track 0.00 -> 79.9 mm, vias 0 -> 1
- net /JTAG_TDI: track 0.00 -> 72.8 mm, vias 0 -> 1
- net /JTAG_TDO: track 0.00 -> 67.1 mm, vias 0 -> 1
- net /CTS0/SCK/TCK: track 0.00 -> 60.8 mm, vias 0 -> 1
- net /DSR0/CS0/TMS: track 0.00 -> 56.1 mm, vias 0 -> 1
- net /DCD0/IO4: track 0.00 -> 39.8 mm, vias 0 -> 1
- net /DTR1: track 0.00 -> 38.9 mm, vias 0 -> 1
- net /I2C_SDA: track 0.00 -> 36.1 mm, vias 0 -> 1
- net /I2C_SCL: track 0.00 -> 36.0 mm, vias 0 -> 1
- net /RXD1: track 0.00 -> 29.7 mm, vias 0 -> 1
- net /USB_Data-: track 0.00 -> 29.6 mm
- net GND: track 0.00 -> 28.9 mm, vias 0 -> 40
- net /USB_Data+: track 0.00 -> 28.3 mm, vias 0 -> 2
- net /RTS1/IO7: track 0.00 -> 28.0 mm, vias 0 -> 1
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- added copper zone on B.Cu, net GND
- added copper zone on F.Cu, net GND
Other:
- board text added: "排针P1 排针P2 工作模式 高电平 高电平 UART1 + UART0 低电平 高电平 UART1 + SPI + I2C (VCP) 高电平 低电平 UART1 + SPI + I2C (HID) 低电平 低电平 UART1 + JTAG"
- board text added: "电子技术博客"

Commit message: Complete PCB wiring.
Routing:
- net /DCD0/IO4: track 39.8 -> 39.1 mm
- net GND: vias 40 -> 39
Other:
- board text added: "UINIO-USB-Serial 串行协议转换器"
- board text removed: "UINIO-USB-Serial"
- board text removed: "电子技术博客"
