File: UINIO-USB-Serial.kicad_pcb (KiCad board)
At the start: 2 copper layers, 55.3 x 28.1 mm, 33 parts, among them J1 Conn_01x07_Pin, J2 Conn_01x10_Pin, J3 Conn_01x04_Pin, J4 Conn_01x07_Pin, J5 排针1, J6 排针2, J7 Conn_01x07_Pin, U1 CH347T, U2 ME6211C33M5G, Y1 8MHz

Commit message: Release UINIO-USB-Serial version 1.0.0.
Parts:
- J5: value 排针1 -> 排针P1
- J6: value 排针2 -> 排针P2
Connections:
- J7 pad 1: GND -> /VDD_3.3V
- J7 pad 7: /VDD_3.3V -> GND
Routing:
- net /VDD_3.3V: track 149.9 -> 138.5 mm

Commit message: Release UINIO-USB-Serial version 1.0.0.
Other:
- board text added: "I2C"
- board text added: "JTAG"
- board text added: "SPI"
- board text added: "UART0"
- board text added: "UART1"
