File: UINIO-USB-Serial.kicad_sch (KiCad schematic)
At the start: 0 parts

Commit message: Finish CH347 core board schema.
Parts:
- added C1, C2: 1uF, Capacitor_SMD:C_0402_1005Metric, symbol Device:C
- added C3, C4, C5, C6: 0.1uF, symbol Device:C
- added D1: LED_Red, LED_SMD:LED_0603_1608Metric, symbol Device:LED
- added D2: LED Blue, symbol Device:LED
- added J1, J2: Conn_01x03_Pin, symbol Connector:Conn_01x03_Pin
- added R1, R2: 5.1K, Resistor_SMD:R_0402_1005Metric, symbol Device:R
- added R3: 2K, Resistor_SMD:R_0402_1005Metric, symbol Device:R
- added R4, R5, R7: 4.7K, symbol Device:R
- added R6: 2K, symbol Device:R
- added U1: ME6211C33M5G-N, Uinio:SOT-23-5_L3.0-W1.7-P0.95-LS2.8-BR, symbol Uinio:ME6211
- added U2: CH347T, Uinio:TSSOP-20_L6.5-W4.4-P0.65-LS6.4-BL, symbol Uinio:CH347T
- added U3: TXS0108EPW, Package_SO:TSSOP-20_4.4x6.5mm_P0.65mm, symbol Logic_LevelTranslator:TXS0108EPW
- added USB1: USB_Type_C_16Pin, Uinio:USB-C-SMD_TYPEC-304J-BCP16, symbol Uinio:USB_Type_C_16Pin
- added Y1: 8MHz, symbol Device:Crystal
Connections:
- new net: C5.2, U2.19 (XI), Y1.1
- new net: C6.2, U2.18 (GND), Y1.2
- new net: D2.2 (A), R6.1
- new net: J2.1 (Pin_1), R7.1
- new net: C3.1, R4.2, U2.1 (RST#)
- new net: D2.1 (K), U2.15 (DCD0/GPIO4/ACT)
- new net: D1.2 (A), R3.1
- new net: J1.1 (Pin_1), R5.1
- new net: R1.1, USB1.A5 (CC1)
- new net: R2.1, USB1.B5 (CC2)
- new net CTS0/SCK/TCK: U2.6 (CTS0/GPIO0/SCK/TCK)
- new net CTS1/IO6: U2.2 (CTS1/GPIO6)
- new net DSR0/CS0/TMS: U2.5 (DSR0/GPIO2/SCS0/TMS)
- new net DTR0/IO5: U2.9 (TNOW0/DTR0/GPIO5/SCS1/TRST)
- new net DTR1: J2.3 (Pin_3), U2.10 (TNOW1/DTR1)
- new net GND: C1.1, C2.1, C3.2, C4.2, C5.1, C6.1, D1.1 (K), R1.2, R2.2, R5.2, R7.2, U1.2 (Vss), USB1.13 (GND), USB1.14 (GND), USB1.15 (GND), USB1.16 (GND), USB1.A1B12 (GND), USB1.B1A12 (GND)
- new net I2C_SCL: U2.11 (RI0/GPIO3/SCL)
- new net I2C_SDA: U2.12 (RXD0/SDA)
- new net JTAG_TDI: U2.8 (TXD0/MOSI/TDI)
- new net JTAG_TDO: U2.7 (RTS0/GPIO1/MISO/TDO)
- new net P1: J1.3 (Pin_3), U2.13 (RTS1/GPIO7)
- new net RXD1: U2.4 (RXD1)
- new net TXD1: U2.3 (TXD1)
- new net USB_Data+: U2.17 (UD+), USB1.A6 (DP1), USB1.B6 (DP2)
- new net USB_Data-: U2.16 (UD-), USB1.A7 (DN1), USB1.B7 (DN2)
- new net VDD_3.3V: C2.2, C4.1, R3.2, R4.1, R6.2, U1.5 (Vout), U2.14 (VCC)
- new net VDD_5V: C1.2, U1.1 (Vin), U1.3 (CE), USB1.A4B9 (VBUS), USB1.B4A9 (VBUS)
- no-connect marks 0 -> 5
Other:
- note added: "I2C"
- note added: "JTAG"
- note added: "OFF"
- note added: "ON"
- note added: "P1 P2 DTR1 RTS1 MODE OFF OFF 1 1 0 ON OFF 1 0 1 OFF ON 0 1 2 ON ON 0 0 3"
- note added: "SPI"
- note added: "UART0"
- note added: "UART1"

Commit message: Update UINIO-USB-Serial schematic diagram.
Parts:
- added C1, C2: 1uF, Capacitor_SMD:C_0402_1005Metric, symbol Device:C
- added D1: LED_Red, LED_SMD:LED_0603_1608Metric, symbol Device:LED
- added J3: Conn_01x03_Pin, symbol Connector:Conn_01x03_Pin
- added J4, J5: Conn_01x16_Pin, symbol Connector:Conn_01x16_Pin
- added R3: 2K, Resistor_SMD:R_0402_1005Metric, symbol Device:R
- added U1: ME6211C18M5G, Uinio:SOT-23-5_L3.0-W1.7-P0.95-LS2.8-BR, symbol Uinio:ME6211
- U1: value ME6211C33M5G-N -> ME6211C33M5G
Connections:
- net CTS0/SCK/TCK: now also J4.10 (Pin_10), J4.3 (Pin_3), J4.5 (Pin_5), J4.6 (Pin_6), J4.7 (Pin_7), J4.8 (Pin_8), J4.9 (Pin_9), J5.13 (Pin_13), J5.5 (Pin_5)
- net CTS1/IO6: now also J4.13 (Pin_13)
- net DSR0/CS0/TMS: now also J5.11 (Pin_11), J5.6 (Pin_6)
- net DTR0/IO5: now also J5.12 (Pin_12), J5.9 (Pin_9)
- net DTR1: now also J4.15 (Pin_15)
- net GND: now also C1.1, C2.1, D1.1 (K), J4.1 (Pin_1), J5.1 (Pin_1), J5.16 (Pin_16), U1.2 (Vss)
- net I2C_SCL: now also J5.3 (Pin_3)
- net I2C_SDA: now also J5.4 (Pin_4)
- net JTAG_TDI: now also J4.4 (Pin_4), J5.15 (Pin_15), J5.7 (Pin_7)
- net JTAG_TDO: now also J5.14 (Pin_14), J5.8 (Pin_8)
- net P1: now also J4.14 (Pin_14)
- net RXD1: now also J4.11 (Pin_11)
- net TXD1: now also J4.12 (Pin_12)
- net VDD_3.3V: now also U3.19 (VCCB), J3.3 (Pin_3), J4.16 (Pin_16), J5.10 (Pin_10)
- net VDD_5V: now also C1.2, J4.2 (Pin_2), J5.2 (Pin_2), U1.1 (Vin), U1.3 (CE)
- net VREF: now reaches U3.10 (OE)
- net VREF: now also U3.2 (VCCA), J3.2 (Pin_2)
- new net: D1.2 (A), R3.1
- new net VDD_1.8V: C2.2, J3.1 (Pin_1), R3.2, U1.5 (Vout)
- no-connect marks 5 -> 7
Other:
- moved on the sheet: U3

Commit message: Complete the schematic test.
Parts:
- removed C1, C2: 1uF, Capacitor_SMD:C_0402_1005Metric, symbol Device:C
- removed D1: LED_Red, LED_SMD:LED_0603_1608Metric, symbol Device:LED
- removed J3: Conn_01x03_Pin, symbol Connector:Conn_01x03_Pin
- removed J4, J5: Conn_01x16_Pin, symbol Connector:Conn_01x16_Pin
- removed R3: 2K, Resistor_SMD:R_0402_1005Metric, symbol Device:R
- removed U1: ME6211C18M5G, Uinio:SOT-23-5_L3.0-W1.7-P0.95-LS2.8-BR, symbol Uinio:ME6211
- removed U3: TXS0108EPW, Package_SO:TSSOP-20_4.4x6.5mm_P0.65mm, symbol Logic_LevelTranslator:TXS0108EPW
- added C? (x3): 0.1uF, Capacitor_SMD:C_0402_1005Metric, symbol Device:C
- added J1: Conn_01x10_Pin, Connector_PinHeader_2.54mm:PinHeader_1x10_P2.54mm_Vertical, symbol Connector:Conn_01x10_Pin
- added J10, J3, J5: Conn_01x07_Pin, Connector_PinHeader_2.54mm:PinHeader_1x07_P2.54mm_Vertical, symbol Connector:Conn_01x07_Pin
- added J2: Conn_01x06_Pin, Connector_PinHeader_2.54mm:PinHeader_1x06_P2.54mm_Vertical, symbol Connector:Conn_01x06_Pin
- added J4, J6, J9: Conn_01x04_Pin, Connector_PinHeader_2.54mm:PinHeader_1x04_P2.54mm_Vertical, symbol Connector:Conn_01x04_Pin
- added R4, R5, R7, R8: 10K, Resistor_SMD:R_0402_1005Metric, symbol Device:R
- added U1: I2C-24-EEPROM-SOIC8, Package_SO:SOIC-8_3.9x4.9mm_P1.27mm, symbol Memory_EEPROM:M24C02-FMN
- added U3: SPI-25-Flash-SOIC8, Package_SO:SOIC-8_5.23x5.23mm_P1.27mm, symbol Memory_Flash:W25Q32JVSS
- added U4: I2C-24-EEPROM-TSSOP8, Package_SO:TSSOP-8_4.4x3mm_P0.65mm, symbol Memory_EEPROM:AT24CS01-XHM
- C1: renamed from C3; footprint (none) -> Capacitor_SMD:C_0402_1005Metric
- C3: renamed from C5; value 0.1uF -> 20pF; footprint (none) -> Capacitor_SMD:C_0402_1005Metric
- C4: renamed from C6; value 0.1uF -> 20pF; footprint (none) -> Capacitor_SMD:C_0402_1005Metric
- C5: renamed from C4; footprint (none) -> Capacitor_SMD:C_0402_1005Metric
- C?: renamed from C1; footprint Capacitor_SMD:C_0402_1005Metric -> Capacitor_SMD:C_0603_1608Metric
- C?: renamed from C2; footprint Capacitor_SMD:C_0402_1005Metric -> Capacitor_SMD:C_0603_1608Metric
- D1: renamed from D2; footprint (none) -> LED_SMD:LED_0603_1608Metric
- J7: renamed from J1; footprint (none) -> Connector_PinHeader_2.54mm:PinHeader_1x03_P2.54mm_Vertical
- J8: renamed from J2; footprint (none) -> Connector_PinHeader_2.54mm:PinHeader_1x03_P2.54mm_Vertical
- R1: renamed from R4; footprint (none) -> Resistor_SMD:R_0402_1005Metric
- R10: renamed from R5; footprint (none) -> Resistor_SMD:R_0402_1005Metric
- R11: renamed from R7; footprint (none) -> Resistor_SMD:R_0402_1005Metric
- R6: footprint (none) -> Resistor_SMD:R_0402_1005Metric
- Y1: footprint (none) -> Crystal:Crystal_SMD_3225-4Pin_3.2x2.5mm
- renumbered D1 to D?, R3 to R?, R1 to R?, R2 to R?, U1 to U?, USB1 to USB?
Connections:
- net CTS0/SCK/TCK: now also J1.2 (Pin_2), J10.2 (Pin_2), J5.4 (Pin_4)
- net CTS1/IO6: now also J3.2 (Pin_2)
- net DSR0/CS0/TMS: now also J1.7 (Pin_7), J10.3 (Pin_3), J5.2 (Pin_2)
- net DTR0/IO5: now also J1.6 (Pin_6), J10.6 (Pin_6), J5.3 (Pin_3)
- net DTR1: now also J8.2 (Pin_2), J3.6 (Pin_6); no longer J8.3 (Pin_3)
- net GND: now also U2.18 (GND), J1.1 (Pin_1), J10.1 (Pin_1), J3.1 (Pin_1), J5.1 (Pin_1), J6.4 (Pin_4)
- net I2C_SCL: now also J1.8 (Pin_8), J6.3 (Pin_3)
- net I2C_SDA: now also J1.4 (Pin_4), J6.2 (Pin_2)
- net JTAG_TDI: now also J1.3 (Pin_3), J10.4 (Pin_4), J5.6 (Pin_6)
- net JTAG_TDO: now also J1.5 (Pin_5), J10.5 (Pin_5), J5.5 (Pin_5)
- net P1: now also J7.2 (Pin_2), J3.5 (Pin_5); no longer J7.3 (Pin_3)
- net RXD1: now also J3.4 (Pin_4)
- net TXD1: now also J3.3 (Pin_3)
- net VDD_3.3V: now also J1.10 (Pin_10), J10.7 (Pin_7), J3.7 (Pin_7), J5.7 (Pin_7), J6.1 (Pin_1)
- net at C3.2, Y1.1: now also U2.20 (XO); no longer U2.19 (XI)
- net at C4.2, Y1.2: now also U2.19 (XI); no longer U2.18 (GND)
- net DCD0/IO4: now reaches D1.1 (K), U2.15 (DCD0/GPIO4/ACT)
- net DCD0/IO4: now also J1.9 (Pin_9)
- new net: J4.3 (Pin_3), R4.1, U1.6 (SCL)
- new net: J9.2 (Pin_2), R8.1, U4.5 (SDA)
- new net: J9.3 (Pin_3), R7.1, U4.6 (SCL)
- new net: J4.2 (Pin_2), R5.1, U1.5 (SDA)
- new net EEPROM-SOIC8-3.3V: C?.2, J4.1 (Pin_1), R4.2, R5.2, U1.8 (VCC)
- new net EEPROM-SOIC8-GND: C?.1, J4.4 (Pin_4), U1.1 (E0), U1.2 (E1), U1.3 (E2), U1.4 (VSS), U1.7 (~{WC})
- new net EEPROM-TSSOP8-3.3V: C?.2, J9.1 (Pin_1), R7.2, R8.2, U4.8 (VCC)
- new net EEPROM-TSSOP8-GND: C?.1, J9.4 (Pin_4), U4.1 (A0), U4.2 (A1), U4.3 (A2), U4.4 (GND), U4.7 (WP)
- new net Flash-SOIC8-3.3V: C?.2, J2.6 (Pin_6), U3.3 (IO2), U3.7 (IO3), U3.8 (VCC)
- new net Flash-SOIC8-CLK: J2.4 (Pin_4), U3.6 (CLK)
- new net Flash-SOIC8-CS: J2.5 (Pin_5), U3.1 (~{CS})
- new net Flash-SOIC8-GND: C?.1, J2.1 (Pin_1), U3.4 (GND)
- new net Flash-SOIC8-MISO: J2.2 (Pin_2), U3.2 (DO(IO1))
- new net Flash-SOIC8-MOSI: J2.3 (Pin_3), U3.5 (DI(IO0))
- no-connect marks 7 -> 5
Other:
- note added: "P1 P2 DTR1 RTS1 MODE OFF OFF 1 1 0 ON OFF 0 1 1 OFF ON 1 0 2 ON ON 0 0 3"
- note removed: "I2C"
- note removed: "JTAG"
- note removed: "P1 P2 DTR1 RTS1 MODE OFF OFF 1 1 0 ON OFF 1 0 1 OFF ON 0 1 2 ON ON 0 0 3"
- note removed: "SPI"
- note removed: "UART0"
- note removed: "UART1"
- moved on the sheet: C1, C3, C4, C5, C?, D1, D?, J7, J8, R1, R10, R11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

Commit message: Finish PCB layout.
Parts:
- removed C3, C4: 20pF, Capacitor_SMD:C_0402_1005Metric, symbol Device:C
- removed C? (x3): 0.1uF, Capacitor_SMD:C_0402_1005Metric, symbol Device:C
- removed J2: Conn_01x06_Pin, Connector_PinHeader_2.54mm:PinHeader_1x06_P2.54mm_Vertical, symbol Connector:Conn_01x06_Pin
- removed J4, J9: Conn_01x04_Pin, Connector_PinHeader_2.54mm:PinHeader_1x04_P2.54mm_Vertical, symbol Connector:Conn_01x04_Pin
- removed R4, R5, R7: 10K, Resistor_SMD:R_0402_1005Metric, symbol Device:R
- removed U1: I2C-24-EEPROM-SOIC8, Package_SO:SOIC-8_3.9x4.9mm_P1.27mm, symbol Memory_EEPROM:M24C02-FMN
- removed U3: SPI-25-Flash-SOIC8, Package_SO:SOIC-8_5.23x5.23mm_P1.27mm, symbol Memory_Flash:W25Q32JVSS
- removed U4: I2C-24-EEPROM-TSSOP8, Package_SO:TSSOP-8_4.4x3mm_P0.65mm, symbol Memory_EEPROM:AT24CS01-XHM
- removed Y1: 8MHz, Crystal:Crystal_SMD_3225-4Pin_3.2x2.5mm, symbol Device:Crystal
- added C? (x2): 20pF, Capacitor_SMD:C_0402_1005Metric, symbol Device:C
- added R9: 4.7K, Resistor_SMD:R_0402_1005Metric, symbol Device:R
- added Y?: 8MHz, Crystal:Crystal_SMD_3225-4Pin_3.2x2.5mm, symbol Device:Crystal_GND24
- J5: renamed from J7; value Conn_01x03_Pin -> 排针1
- J6: renamed from J8; value Conn_01x03_Pin -> 排针2
- R8: value 10K -> 4.7K
- R? (x2): footprint Resistor_SMD:R_0402_1005Metric -> Resistor_SMD:R_0603_1608Metric
- renumbered C5 to C3, J5 to J1, J1 to J2, J6 to J3, J3 to J4, J10 to J7, R6 to R4, R10 to R6, R11 to R7, U2 to U1
Connections:
- net EEPROM-TSSOP8-3.3V is gone; now on net VDD_3.3V: R8.2
- net CTS0/SCK/TCK: now also J2.4 (Pin_4); no longer J2.2 (Pin_2)
- net CTS1/IO6: now also J4.4 (Pin_4); no longer J4.2 (Pin_2)
- net GND: now also C?.1, C?.1, Y?.2, Y?.4
- net I2C_SDA: now also J2.3 (Pin_3); no longer J2.4 (Pin_4)
- net JTAG_TDI: now also J2.2 (Pin_2); no longer J2.3 (Pin_3)
- net RXD1: now also J4.3 (Pin_3); no longer J4.4 (Pin_4)
- net TXD1: now also J4.2 (Pin_2); no longer J4.3 (Pin_3)
- net VDD_3.3V: now also R9.2
- net at U1.20 (XO): now also C?.2, Y?.1
- net at U1.19 (XI): now also C?.2, Y?.3
- net at R8.1: now also J5.3 (Pin_3)
- net at J6.3 (Pin_3): now also R9.1
- net P1 renamed RTS1/IO7
- no-connect marks 5 -> 3
Other:
- note added: "P1 P2 DTR1 RTS1 MODE 高电平 高电平 1 1 0 低电平 高电平 0 1 1 高电平 低电平 1 0 2 低电平 低电平 0 0 3"
- note added: "上拉"
- note added: "下拉"
- note removed: "OFF"
- note removed: "ON"
- note removed: "P1 P2 DTR1 RTS1 MODE OFF OFF 1 1 0 ON OFF 0 1 1 OFF ON 1 0 2 ON ON 0 0 3"
- moved on the sheet: J1, J2, J3, J4, J5, J6, J7, R6, R7, R?, USB?

Commit message: Finish PCB layout.
Parts:
- J5: value 排针1 -> 排针P1
- J6: value 排针2 -> 排针P2
Connections:
- net CTS0/SCK/TCK: now also J1.3 (Pin_3), J2.5 (Pin_5), J7.3 (Pin_3); no longer J1.4 (Pin_4), J2.4 (Pin_4), J7.2 (Pin_2)
- net CTS1/IO6: now also J4.3 (Pin_3); no longer J4.4 (Pin_4)
- net DCD0/IO4: now also J2.7 (Pin_7); no longer J2.9 (Pin_9)
- net DSR0/CS0/TMS: now also J2.6 (Pin_6), J7.2 (Pin_2); no longer J2.7 (Pin_7), J7.3 (Pin_3)
- net DTR0/IO5: now also J1.6 (Pin_6), J2.2 (Pin_2); no longer J1.3 (Pin_3), J2.6 (Pin_6)
- net I2C_SCL: now also J2.9 (Pin_9), J3.2 (Pin_2); no longer J2.8 (Pin_8), J3.3 (Pin_3)
- net I2C_SDA: now also J2.8 (Pin_8), J3.3 (Pin_3); no longer J2.3 (Pin_3), J3.2 (Pin_2)
- net JTAG_TDI: now also J1.5 (Pin_5), J2.3 (Pin_3), J7.5 (Pin_5); no longer J1.6 (Pin_6), J2.2 (Pin_2), J7.4 (Pin_4)
- net JTAG_TDO: now also J1.4 (Pin_4), J2.4 (Pin_4), J7.4 (Pin_4); no longer J1.5 (Pin_5), J2.5 (Pin_5), J7.5 (Pin_5)
- net RTS1/IO7: now also J4.2 (Pin_2); no longer J4.5 (Pin_5)
- net RXD1: now also J4.5 (Pin_5); no longer J4.3 (Pin_3)
- net TXD1: now also J4.4 (Pin_4); no longer J4.2 (Pin_2)
Other:
- note added: "排针P1 排针P2 DTR1 RTS1 MODE 高电平 高电平 1 1 0 低电平 高电平 0 1 1 高电平 低电平 1 0 2 低电平 低电平 0 0 3"
- note removed: "P1 P2 DTR1 RTS1 MODE 高电平 高电平 1 1 0 低电平 高电平 0 1 1 高电平 低电平 1 0 2 低电平 低电平 0 0 3"

Commit message: Release UINIO-USB-Serial version 1.0.0.
Other:
- company: 电子技术博客 UinIO.com -> UinIO.com 硬件电子实验室
Changed lines of the file:
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@@
     (date "2023-12-26")
     (rev "Version 1.0.0")
-    (company "电子技术博客 UinIO.com")
+    (company "UinIO.com 硬件电子实验室")
   )
   (junction (at 157.48 97.79) (diameter 0) (color 0 0 0 0)

Commit message: Release UINIO-USB-Serial version 1.0.0.
Connections:
- net GND: now also J7.7 (Pin_7); no longer J7.1 (Pin_1)
- net VDD_3.3V: now also J7.1 (Pin_1); no longer J7.7 (Pin_7)
Other:
- company: UinIO.com 硬件电子实验室 -> UinIO.com 电子技术实验室
Changed lines of the file:
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@@
   (title_block
     (title "UINIO-USB-Serial")
-    (date "2023-12-26")
+    (date "2024-01-09")
     (rev "Version 1.0.0")
-    (company "UinIO.com 硬件电子实验室")
+    (company "UinIO.com 电子技术实验室")
   )
   (junction (at 157.48 97.79) (diameter 0) (color 0 0 0 0)
@@
     (stroke (width 0) (type default))
   )
-  (wire (pts (xy 262.89 168.91) (xy 264.16 168.91))
+  (wire (pts (xy 262.89 184.15) (xy 264.16 184.15))
     (stroke (width 0) (type default))
   )
@@
     (stroke (width 0) (type default))
   )
-  (wire (pts (xy 261.62 184.15) (xy 264.16 184.15))
+  (wire (pts (xy 261.62 168.91) (xy 264.16 168.91))
     (stroke (width 0) (type default))
   )
@@
     (effects (font (size 1.27 1.27)) (justify left bottom))
   )
-  (label "VDD_3.3V" (at 261.62 184.15 180) (fields_autoplaced)
+  (label "VDD_3.3V" (at 261.62 168.91 180) (fields_autoplaced)
     (effects (font (size 1.27 1.27)) (justify right bottom))
   )
@@
     )
   )
-  (symbol (lib_id "power:GND") (at 262.89 168.91 270) (unit 1)
-    (in_bom yes) (on_board yes) (dnp no)
-    (property "Reference" "#PWR?" (at 256.54 168.91 0)
-      (effects (font (size 1.27 1.27)) hide)
-    )
-    (property "Value" "GND" (at 258.445 167.64 90)
-      (effects (font (size 1.27 1.27)))
-    )
-    (property "Footprint" "" (at 262.89 168.91 0)
-      (effects (font (size 1.27 1.27)) hide)
-    )
-    (property "Datasheet" "" (at 262.89 168.91 0)
-      (effects (font (size 1.27 1.27)) hide)
-    )
+  (symbol (lib_id "power:GND") (at 262.89 184.15 270) (unit 1)
+    (in_bom yes) (on_board yes) (dnp no)
+    (property "Reference" "#PWR?" (at 256.54 184.15 0)
+      (effects (font (size 1.27 1.27)) hide)
+    )
+    (property "Value" "GND" (at 257.81 184.15 90)
+      (effects (font (size 1.27 1.27)))
+    )
+    (property "Footprint" "" (at 262.89 184.15 0)
+      (effects (font (size 1.27 1.27)) hide)
+    )
+    (property "Datasheet" "" (at 262.89 184.15 0)
+      (effects (font (size 1.27 1.27)) hide)
+    )
